File: Relaisplatine_I2C.kicad_sch (KiCad schematic)
At the start: 78 parts, among them J1 K, J1.1 G1-K, J1.1a1001 G1-J, J1.1a1002 G1-K, J1.1a1003 G1-K, J1.1a1004 G1-K, J1.1a1005 G1-K, J1.1a1006 G1-K, J1.1a1007 G1-K, J1.2 G1-J, J1.2a1001 G1-K, J1.2a1002 G1-J, J1.2a1003 G1-J, J1.2a1004 G1-J, J1.2a1005 G1-J, J1.2a1006 G1-J, J1.2a1007 G1-J, J10 I²C, J11 Relais-Power, J12 Int, J2 J, J2.1 G2-K, J2.1a1001 G1-J, J2.2 G2-J, J2.2a1001 G2-K, J3.1 G3-K, J3.2 G3-J, J4.1 G4-K, J4.2 G4-J, J5.1 G5-K, J5.2 G5-J, J6.1 G6-K, J6.2 G6-J, J7.1 G7-K, J7.2 G7-J, J8.1 G8-K, J8.2 G8-J, U1 ULN2803A, U2 PCF8574

Commit message: Abstand Fläche - Plarineneand auf 1mm gesetzt
Parts:
- A0, A1, A2: footprint Jumper:SolderJumper-3_P1.3mm_Bridged12_Pad1.0x1.5mm_NumberLabels -> Jumper:SolderJumper-3_P1.3mm_Open_RoundedPad1.0x1.5mm
Changed lines of the file:
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@@
       (effects (font (size 1.27 1.27)) (justify left) hide)
     )
-    (property "Footprint" "Jumper:SolderJumper-3_P1.3mm_Bridged12_Pad1.0x1.5mm_NumberLabels" (at 63.5 129.54 0)
+    (property "Footprint" "Jumper:SolderJumper-3_P1.3mm_Open_RoundedPad1.0x1.5mm" (at 63.5 129.54 0)
       (effects (font (size 1.27 1.27)) hide)
     )
@@
       (effects (font (size 1.27 1.27)) (justify left) hide)
     )
-    (property "Footprint" "Jumper:SolderJumper-3_P1.3mm_Bridged12_Pad1.0x1.5mm_NumberLabels" (at 77.47 135.89 0)
+    (property "Footprint" "Jumper:SolderJumper-3_P1.3mm_Open_RoundedPad1.0x1.5mm" (at 77.47 135.89 0)
       (effects (font (size 1.27 1.27)) hide)
     )
@@
       (effects (font (size 1.27 1.27)) (justify left) hide)
     )
-    (property "Footprint" "Jumper:SolderJumper-3_P1.3mm_Bridged12_Pad1.0x1.5mm_NumberLabels" (at 71.12 133.35 0)
-      (effects (font (size 1.27 1.27)) hide)
-    )
+    (property "Footprint" "Jumper:SolderJumper-3_P1.3mm_Open_RoundedPad1.0x1.5mm" (at 71.12 133.35 0)
+      (effects (font (size 1.27 1.27)) hide)
+    )

Commit message: Kosmetik
Parts:
- RN1: value RN1 -> 680
- RN2: value R_Network04 -> 680
Other:
- note added: "PCF8574P : 0x20-0x27 PCF8574AP: 0x38-0x3f"
